File: Hardware/AK9750 Human Movement Sensor Breakout.brd (EAGLE design)
At the start: 25.4 x 25.4 mm, 26 parts, among them J2 SMD, J3 PTH, J4 SMD, U2 AK9750

Commit message: Adding panel files
Parts:
- moved JP3 1.80 mm to (3.81, 21.6)
- moved JP4 1.80 mm to (21.6, 21.6)
Routing:
- net 3.3V: track 78.2 -> 77.7 mm
Other:
- board text added: "X11"
- board text removed: "X01"
